File: max660_invertor.kicad_sch (KiCad schematic)
At the start: 5 parts, among them U1 MAX660

Commit message: add image
Parts:
- H1: value ~ -> -5v
- H2: value ~ -> +5v
Connections:
- net +5V: no longer names the net of H2.1, U1.8 (VIN)
- net -5V: no longer names the net of C2.2, H1.1, U1.5 (SHDN)
